Commit message: Rely on package instead of searching for specific files

File: husky_description/urdf/decorations.urdf.xacro (robot description, xacro)
@@ -1,11 +1,26 @@
 <?xml version="1.0"?>
-<robot name="husky_decorations" xmlns:xacro="http://ros.org/wiki/xacro">
-  <material name="dark_grey"><color rgba="0.2 0.2 0.2 1.0" /></material>
-  <material name="medium_grey"><color rgba="0.6 0.6 0.6 1.0" /></material>
-  <material name="light_grey"><color rgba="0.8 0.8 0.8 1.0" /></material>
-  <material name="yellow"><color rgba="0.8 0.8 0.0 1.0" /></material>
-  <material name="black"><color rgba="0.15 0.15 0.15 1.0" /></material>
-  <material name="white"><color rgba="1.0 1.0 1.0 1.0" /></material>
-  <material name="red"><color rgba="1.0 0.0 0.0 1.0" /></material>
+<robot name="husky_decorations"
+  xmlns:xacro="http://ros.org/wiki/xacro">
+  <material name="dark_grey">
+    <color rgba="0.2 0.2 0.2 1.0" />
+  </material>
+  <material name="medium_grey">
+    <color rgba="0.6 0.6 0.6 1.0" />
+  </material>
+  <material name="light_grey">
+    <color rgba="0.8 0.8 0.8 1.0" />
+  </material>
+  <material name="yellow">
+    <color rgba="0.8 0.8 0.0 1.0" />
+  </material>
+  <material name="black">
+    <color rgba="0.15 0.15 0.15 1.0" />
+  </material>
+  <material name="white">
+    <color rgba="1.0 1.0 1.0 1.0" />
+  </material>
+  <material name="red">
+    <color rgba="1.0 0.0 0.0 1.0" />
+  </material>
   <xacro:macro name="husky_decorate">
     <xacro:property name="husky_front_bumper_extend" value="$(optenv HUSKY_FRONT_BUMPER_EXTEND 0)" />
@@ -16,5 +31,5 @@
         <origin xyz="0 0 0" rpy="0 0 0" />
         <geometry>
-          <mesh filename="file://$(find husky_description)/meshes/top_chassis.dae" />
+          <mesh filename="package://husky_description/meshes/top_chassis.dae" />
         </geometry>
       </visual>
@@ -30,5 +45,5 @@
         <visual>
           <geometry>
-            <mesh filename="file://$(find husky_description)/meshes/user_rail.dae" />
+            <mesh filename="package://husky_description/meshes/user_rail.dae" />
           </geometry>
         </visual>
@@ -45,5 +60,5 @@
       <visual>
         <geometry>
-          <mesh filename="file://$(find husky_description)/meshes/bumper.dae" />
+          <mesh filename="package://husky_description/meshes/bumper.dae" />
         </geometry>
       </visual>
@@ -57,9 +72,9 @@
     <xacro:if value="${husky_front_bumper_extend}">
       <link name="front_bumper_extension_link">
-          <visual>
-              <geometry>
-                  <mesh filename="file://$(find husky_description)/meshes/bumper_extension.dae" />
-              </geometry>
-          </visual>
+        <visual>
+          <geometry>
+            <mesh filename="package://husky_description/meshes/bumper_extension.dae" />
+          </geometry>
+        </visual>
       </link>
       <joint name="front_bumper_extension" type="fixed">
@@ -73,5 +88,5 @@
       <visual>
         <geometry>
-          <mesh filename="file://$(find husky_description)/meshes/bumper.dae" />
+          <mesh filename="package://husky_description/meshes/bumper.dae" />
         </geometry>
       </visual>
@@ -85,9 +100,9 @@
     <xacro:if value="${husky_rear_bumper_extend}">
       <link name="rear_bumper_extension_link">
-          <visual>
-              <geometry>
-                  <mesh filename="file://$(find husky_description)/meshes/bumper_extension.dae" />
-              </geometry>
-          </visual>
+        <visual>
+          <geometry>
+            <mesh filename="package://husky_description/meshes/bumper_extension.dae" />
+          </geometry>
+        </visual>
       </link>
       <joint name="rear_bumper_extension" type="fixed">
@@ -104,5 +119,5 @@
             <origin xyz="0 0 0" rpy="0 0 0" />
             <geometry>
-              <mesh filename="file://$(find husky_description)/meshes/large_top_plate.dae" />
+              <mesh filename="package://husky_description/meshes/large_top_plate.dae" />
             </geometry>
           </visual>
@@ -110,5 +125,5 @@
             <origin xyz="0 0 0" rpy="0 0 0"/>
             <geometry>
-              <mesh filename="file://$(find husky_description)/meshes/large_top_plate_collision.stl" />
+              <mesh filename="package://husky_description/meshes/large_top_plate_collision.stl" />
             </geometry>
           </collision>
@@ -138,5 +153,5 @@
             <origin xyz="0 0 0" rpy="0 0 0" />
             <geometry>
-              <mesh filename="file://$(find husky_description)/meshes/top_plate.dae" />
+              <mesh filename="package://husky_description/meshes/top_plate.dae" />
             </geometry>
           </visual>
@@ -144,5 +159,5 @@
             <origin xyz="0 0 0" rpy="0 0 0"/>
             <geometry>
-              <mesh filename="file://$(find husky_description)/meshes/top_plate.stl" />
+              <mesh filename="package://husky_description/meshes/top_plate.stl" />
             </geometry>
           </collision>

File: husky_description/urdf/husky_macro.urdf.xacro (robot description, xacro)
@@ -37,5 +37,5 @@
         <origin xyz="0 0 0" rpy="0 0 0" />
         <geometry>
-          <mesh filename="file://$(find husky_description)/meshes/base_link.dae" />
+          <mesh filename="package://husky_description/meshes/base_link.dae" />
         </geometry>
       </visual>
@@ -154,5 +154,5 @@
           <param name="max_speed">1.0</param>
           <param name="polling_timeout">10.0</param>
-	  <param name="serial_port">/dev/serial/by-id/usb-FTDI_FT232R_USB_UART_A6031ITX-if00-port0</param>
+          <param name="serial_port">/dev/serial/by-id/usb-FTDI_FT232R_USB_UART_A6031ITX-if00-port0</param>
         </xacro:unless>
       </hardware>

File: husky_description/urdf/wheel.urdf.xacro (robot description, xacro)
@@ -6,10 +6,10 @@
         <mass value="2.637" />
         <origin xyz="0 0 0" />
-        <inertia  ixx="0.02467" ixy="0" ixz="0" iyy="0.04411" iyz="0" izz="0.02467" />
+        <inertia ixx="0.02467" ixy="0" ixz="0" iyy="0.04411" iyz="0" izz="0.02467" />
       </inertial>
       <visual>
         <origin xyz="0 0 0" rpy="0 0 0" />
         <geometry>
-          <mesh filename="file://$(find husky_description)/meshes/wheel.dae" />
+          <mesh filename="package://husky_description/meshes/wheel.dae" />
         </geometry>
       </visual>

Commit message: Hide top plate in Husky description

File: husky_description/urdf/decorations.urdf.xacro (robot description, xacro)
@@ -150,16 +150,16 @@
       <xacro:unless value="$(optenv HUSKY_LARGE_TOP_PLATE false)">
         <link name="top_plate_link">
-          <visual>
+          <!-- <visual>
             <origin xyz="0 0 0" rpy="0 0 0" />
             <geometry>
               <mesh filename="package://husky_description/meshes/top_plate.dae" />
             </geometry>
-          </visual>
-          <collision>
+          </visual> -->
+          <!-- <collision>
             <origin xyz="0 0 0" rpy="0 0 0"/>
             <geometry>
               <mesh filename="package://husky_description/meshes/top_plate.stl" />
             </geometry>
-          </collision>
+          </collision> -->
         </link>
         <!-- Attach top plate -->

Commit message: Launch robot description in base_launch the same way as marmotte_description

File: husky_description/urdf/decorations.urdf.xacro (robot description, xacro)
@@ -116,16 +116,16 @@
       <xacro:if value="$(optenv HUSKY_LARGE_TOP_PLATE false)">
         <link name="top_plate_link">
-          <visual>
+          <!-- <visual>
             <origin xyz="0 0 0" rpy="0 0 0" />
             <geometry>
               <mesh filename="package://husky_description/meshes/large_top_plate.dae" />
             </geometry>
-          </visual>
-          <collision>
+          </visual> -->
+          <!-- <collision>
             <origin xyz="0 0 0" rpy="0 0 0"/>
             <geometry>
               <mesh filename="package://husky_description/meshes/large_top_plate_collision.stl" />
             </geometry>
-          </collision>
+          </collision> -->
         </link>
         <!-- Attach top plate -->
